Commit message: Got the joint state publisher working!

File: urdf/rrbot.xacro (robot description, xacro)
@@ -155,14 +155,4 @@
     </actuator>
   </transmission>
-  <transmission name="tran1">
-    <type>transmission_interface/SimpleTransmission</type>
-    <joint name="joint1">
-      <hardwareInterface>hardware_interface/EffortJointInterface</hardwareInterface>
-    </joint>
-    <actuator name="motor1">
-      <hardwareInterface>hardware_interface/EffortJointInterface</hardwareInterface>
-      <mechanicalReduction>1</mechanicalReduction>
-    </actuator>
-  </transmission>
   <transmission name="tran2">
     <type>transmission_interface/SimpleTransmission</type>
@@ -175,5 +165,5 @@
     </actuator>
   </transmission>
- <transmission name="tran2">
+ <transmission name="prismatic">
     <type>transmission_interface/SimpleTransmission</type>
     <joint name="prismatic">

Commit message: PID integration - still needs IK

File: urdf/rrbot.xacro (robot description, xacro)
@@ -4,5 +4,5 @@
   <!-- Constants for robot dimensions -->
   <xacro:property name="PI" value="3.1415926535897931"/>
-  <xacro:property name="mass" value="1" /> <!-- arbitrary value for mass -->
+  <xacro:property name="mass" value=".01" /> <!-- arbitrary value for mass -->
   <xacro:property name="width" value="0.1" /> <!-- Square dimensions (widthxwidth) of beams -->
   <xacro:property name="height1" value="1" /> <!-- Link 1 -->
@@ -18,7 +18,8 @@
   <!-- Used for fixing robot to Gazebo 'base_link' -->
   <link name="world"/>
-  <joint name="joint0" type="continuous">
+  <joint name="joint0" type="revolute">
     <parent link="world"/>
     <child link="link1"/>
+    <limit effort="1000.0" lower="-3.14159" upper="3.14159" velocity="10"/>
     <origin xyz="0 0 0" rpy="0 0 0"/>
     <axis xyz="0 0 1"/>
@@ -44,7 +45,7 @@
       <mass value="${mass}"/>
       <inertia
-	  ixx="${mass / 12.0 * (width*width + height1*height1)}" ixy="0.0" ixz="0.0"
-	  iyy="${mass / 12.0 * (height1*height1 + width*width)}" iyz="0.0"
-	  izz="${mass / 12.0 * (width*width + width*width)}"/>
+	  ixx="${0}" ixy="0.0" ixz="0.0"
+	  iyy="${0}" iyz="0.0"
+	  izz="${0}"/>
     </inertial>
   </link>
@@ -73,10 +74,11 @@
       <mass value="${mass}"/>
       <inertia
-	  ixx="${mass / 12.0 * (width*width + height2*height2)}" ixy="0.0" ixz="0.0"
-	  iyy="${mass / 12.0 * (height2*height2 + width*width)}" iyz="0.0"
-	  izz="${mass / 12.0 * (width*width + width*width)}"/>
+	  ixx="${0}" ixy="0.0" ixz="0.0"
+	  iyy="${0}" iyz="0.0"
+	  izz="${0}"/>
     </inertial>
   </link>
   <joint name="joint2" type="continuous">
+    <limit effort="1000.0" lower="-3.14159" upper="3.14159" velocity="10"/>
     <parent link="link2"/>
     <child link="link3"/>
@@ -105,7 +107,7 @@
       <mass value="${mass}"/>
       <inertia
-	  ixx="${mass / 12.0 * (width*width + height3*height3)}" ixy="0.0" ixz="0.0"
-	  iyy="${mass / 12.0 * (height3*height3 + width*width)}" iyz="0.0"
-	  izz="${mass / 12.0 * (width*width + width*width)}"/>
+	  ixx="${0}" ixy="0.0" ixz="0.0"
+	  iyy="${0}" iyz="0.0"
+	  izz="${0}"/>
     </inertial>
 	<gravity>0</gravity>
